File: 65-keyboard-pcb.kicad_pcb (KiCad board)
At the start: 2 copper layers, 304.8 x 102.4 mm, 153 parts, among them J1 USB4085-GF-A_REVA, SW1 SW_PUSH, U1 ATmega32U4-AU, X1 XTAL_GND

Commit message: Component placement
Parts:
- U1: value ATmega32U4-AU -> ATMEGA32U4
- moved R4 362.8 mm to (263.8, 48.2), turned to 90 degrees
- moved R5 354.4 mm to (250.6, 48.2), turned to 270 degrees
- moved SW1 335.9 mm to (202.8, 137.3)
- moved F1 320.5 mm to (202.7, 129.1), turned to 180 degrees
- moved R6 300.7 mm to (191.9, 135.5), turned to 180 degrees
- moved R2 286.8 mm to (193.4, 124.8)
- moved R3 281.3 mm to (193.4, 127.0)
- moved C4 274.8 mm to (176.3, 124.8), turned to 180 degrees
- moved C7 272.7 mm to (191.9, 131.2)
- moved C5 271.7 mm to (176.2, 141.6), turned to 180 degrees
- moved C8 270.6 mm to (185.6, 124.8)
- moved C1 264.5 mm to (188.7, 128.0)
- moved C6 260.5 mm to (170.1, 135.5), turned to 180 degrees
- moved R1 257.9 mm to (173.1, 138.6), turned to 180 degrees
- moved C3 19.3 mm to (193.9, 142.5), turned to 270 degrees
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Connections:
- U1 pad 16: XTAL2 -> XTAL1
- U1 pad 17: XTAL1 -> XTAL2
- U1 pad 2: Net-(U1-Pad2) -> +5V
- U1 pad 24: Net-(U1-Pad2) -> +5V
- U1 pad 44: Net-(U1-Pad2) -> +5V
Other:
- outline, holes or cut-outs redrawn

Commit message: Route traces
Parts:
- moved C2 8.76 mm to (193.9, 142.5)
- moved C3 8.76 mm to (185.2, 142.5)
- moved R5 7.33 mm to (255.6, 53.5), turned to 90 degrees
- moved R4 6.11 mm to (260.9, 53.5)
- moved F1 4.36 mm to (198.4, 130.0)
- moved SW1 4.34 mm to (199.3, 134.7), turned to 180 degrees
- turned X1 to 180 degrees
Routing:
- net VCC: track 0.00 -> 145.4 mm
- net Net-(J1-PadA6): track 0.00 -> 138.5 mm, vias 0 -> 2
- net Net-(J1-PadA7): track 0.00 -> 137.1 mm
- net +5V: track 0.00 -> 102.8 mm, vias 0 -> 3
- net GND: track 0.00 -> 41.2 mm
- net RESET: track 0.00 -> 16.6 mm
- net XTAL1: track 0.00 -> 11.5 mm
- net Net-(D7-Pad2): track 0.00 -> 10.8 mm
- net Net-(D15-Pad2): track 0.00 -> 10.8 mm
- net Net-(D4-Pad2): track 0.00 -> 10.8 mm
- net Net-(D20-Pad2): track 0.00 -> 10.8 mm
- net Net-(D2-Pad2): track 0.00 -> 10.8 mm
- net Net-(D8-Pad2): track 0.00 -> 10.8 mm
- net Net-(D13-Pad2): track 0.00 -> 10.8 mm
- net Net-(D3-Pad2): track 0.00 -> 10.8 mm
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Other:
- net class Power added: clearance 0.2, trace_width 0.4, via_dia 0.8, via_drill 0.4

Commit message: Route traces
Parts:
- removed MX62: MX-NoLED, MX_Only:MXOnly-7U-ReversedStabilizers-NoLED
- moved C2 2.59 mm to (191.8, 144.0), turned to 180 degrees
- moved C3 2.59 mm to (187.3, 144.0), turned to 0 degrees
Connections:
- U1 pad 12: Net-(U1-Pad12) -> COL13
- U1 pad 18: Net-(U1-Pad18) -> COL14
- U1 pad 19: Net-(U1-Pad19) -> COL12
- U1 pad 20: Net-(U1-Pad20) -> COL11
- U1 pad 21: Net-(U1-Pad21) -> COL10
- U1 pad 22: Net-(U1-Pad22) -> COL9
- U1 pad 25: Net-(U1-Pad25) -> COL8
- U1 pad 26: Net-(U1-Pad26) -> ROW0
- U1 pad 27: Net-(U1-Pad27) -> ROW1
- U1 pad 28: Net-(U1-Pad28) -> ROW2
- U1 pad 29: Net-(U1-Pad29) -> ROW3
- U1 pad 30: Net-(U1-Pad30) -> ROW4
- U1 pad 31: Net-(U1-Pad31) -> COL6
- U1 pad 32: Net-(U1-Pad32) -> COL5
- U1 pad 36: Net-(U1-Pad36) -> COL4
- U1 pad 37: Net-(U1-Pad37) -> COL3
- U1 pad 38: Net-(U1-Pad38) -> COL2
- U1 pad 39: Net-(U1-Pad39) -> COL1
- U1 pad 40: Net-(U1-Pad40) -> COL0
- U1 pad 41: Net-(U1-Pad41) -> COL7
Routing:
- net ROW4: track 0.00 -> 292.6 mm, vias 0 -> 3
- net ROW0: track 0.00 -> 288.9 mm, vias 0 -> 3
- net COL0: track 0.00 -> 288.9 mm, vias 0 -> 10
- net ROW2: track 0.00 -> 286.4 mm, vias 0 -> 3
- net ROW1: track 0.00 -> 284.0 mm, vias 0 -> 3
- net COL1: track 0.00 -> 280.9 mm, vias 0 -> 10
- net ROW3: track 0.00 -> 276.0 mm, vias 0 -> 3
- net COL2: track 0.00 -> 252.7 mm, vias 0 -> 10
- net COL3: track 0.00 -> 211.1 mm, vias 0 -> 10
- net COL4: track 0.00 -> 188.9 mm, vias 0 -> 10
- net COL6: track 0.00 -> 168.0 mm, vias 0 -> 9
- net COL5: track 0.00 -> 166.8 mm, vias 0 -> 9
- net COL7: track 0.00 -> 131.6 mm, vias 0 -> 10
- net COL12: track 0.00 -> 112.9 mm
- net COL11: track 0.00 -> 98.9 mm
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- added copper zone on B.Cu, net GND
- added copper zone on F.Cu, net GND

Commit message: Route traces
Parts:
- added MX62: MX-NoLED, MX_Only:MXOnly-7U-ReversedStabilizers-NoLED, F.Cu at (147.6, 133.3)
Routing:
- net COL6: track 168.0 -> 217.7 mm, vias 9 -> 8
- net COL5: track 166.8 -> 213.0 mm, vias 9 -> 8
- net COL4: track 188.9 -> 219.1 mm
- net COL2: track 252.7 -> 280.7 mm
- net COL3: track 211.1 -> 237.7 mm
- net COL0: track 288.9 -> 315.2 mm
- net COL1: track 280.9 -> 305.8 mm
- net COL7: track 131.6 -> 154.7 mm
- net VCC: track 145.4 -> 146.5 mm
- net GND: vias 5 -> 8

Commit message: PCB
Parts:
- removed D15, D29, D30, D44, D48, D49, D51, D52, D53, D58, D59, D60, D61, D62, D63, D64, D65, D66, D67: 22p, Diode_SMD:D_SOD-123
- removed MX15, MX30, MX44, MX48, MX49, MX51, MX52, MX53, MX58, MX64, MX65, MX66, MX67: MX-NoLED, MX_Only:MXOnly-1U-NoLED
- removed MX29: MX-NoLED, MX_Only:MXOnly-1.5U-NoLED
- removed MX59, MX60, MX61, MX63: MX-NoLED, MX_Only:MXOnly-1.25U-NoLED
- removed MX62: MX-NoLED, MX_Only:MXOnly-7U-ReversedStabilizers-NoLED
- J1: moved to F.Cu
- MX14: footprint MX_Only:MXOnly-2U-NoLED -> MX_Only:MXOnly-1U-NoLED
- MX16: footprint MX_Only:MXOnly-1.5U-NoLED -> MX_Only:MXOnly-1.25U-NoLED
- MX27: footprint MX_Only:MXOnly-1U-NoLED -> MX_Only:MXOnly-1.75U-NoLED
- MX31: footprint MX_Only:MXOnly-1.25U-NoLED -> MX_Only:MXOnly-1.75U-NoLED
- MX41, MX47, MX54: footprint MX_Only:MXOnly-1U-NoLED -> MX_Only:MXOnly-1.25U-NoLED
- MX43: footprint MX_Only:MXOnly-2.25U-NoLED -> MX_Only:MXOnly-1U-NoLED
- MX45: footprint MX_Only:MXOnly-2.25U-NoLED -> MX_Only:MXOnly-1.25U-NoLED
- MX50: footprint MX_Only:MXOnly-1U-NoLED -> MX_Only:MXOnly-6.25U-ReversedStabilizers-NoLED
- MX56: footprint MX_Only:MXOnly-1.75U-NoLED -> MX_Only:MXOnly-1U-NoLED
- moved R4 232.5 mm to (28.7, 67.1)
- moved R5 225.3 mm to (30.7, 67.1)
- moved J1 209.1 mm to (48.6, 60.1), turned to 180 degrees
- moved F1 164.3 mm to (46.5, 67.5), turned to 270 degrees
- moved R2 155.8 mm to (48.8, 67.1), turned to 90 degrees
- moved R3 154.7 mm to (50.8, 67.1), turned to 90 degrees
- moved C2 103.3 mm to (90.7, 122.7), turned to 90 degrees
- moved X1 96.5 mm to (94.7, 122.8)
- moved C1 95.8 mm to (93.0, 128.1)
- moved C3 89.7 mm to (100.7, 120.8)
- moved C7 87.0 mm to (105.5, 120.8)
- moved C8 86.1 mm to (100.7, 139.2)
- moved SW1 80.8 mm to (120.2, 151.3)
- moved U1 77.9 mm to (103.1, 129.5), turned to 45 degrees
- moved C6 77.2 mm to (93.0, 130.9), turned to 0 degrees
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Connections:
- U1 pad 18: COL14 -> Net-(U1-Pad18)
- U1 pad 30: ROW4 -> Net-(U1-Pad30)
- X1 pad 2: XTAL2 -> GND
- X1 pad 3: GND -> XTAL2
- X1 pad 4: (no net) -> GND
Routing:
- net COL0: track 315.2 -> 0.00 mm, vias 10 -> 0
- net COL1: track 305.8 -> 0.00 mm, vias 10 -> 0
- net ROW4: track 292.6 -> 0.00 mm, vias 3 -> 0
- net COL2: track 280.7 -> 0.00 mm, vias 10 -> 0
- net COL3: track 237.7 -> 0.00 mm, vias 10 -> 0
- net COL4: track 219.1 -> 0.00 mm, vias 10 -> 0
- net COL6: track 217.7 -> 0.00 mm, vias 8 -> 0
- net COL5: track 213.0 -> 0.00 mm, vias 8 -> 0
- net COL7: track 154.7 -> 0.00 mm, vias 10 -> 0
- net VCC: track 146.5 -> 9.62 mm
- net Net-(J1-PadA6): track 138.5 -> 4.41 mm, vias 2 -> 0
- net Net-(J1-PadA7): track 137.1 -> 3.72 mm
- net +5V: track 113.7 -> 0.07 mm, vias 5 -> 0
- net COL12: track 112.9 -> 0.00 mm
- net GND: track 120.3 -> 13.1 mm, vias 8 -> 0
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- removed copper zone on B.Cu, net GND
- removed copper zone on F.Cu, net GND
Other:
- board size 304.8 x 102.4 mm -> 276.2 x 85.7 mm
- board text added: "Keyboar"
