File: 65-keyboard-pcb.sch (KiCad schematic (older format))
At the start: 67 parts

Commit message: Design matrix
Parts:
- added D? (x67): 22p, symbol Device:D_Small
Connections:
- net COL3: now reaches MX?.1 (COL)
- net COL3: now also MX?.1 (COL), MX?.1 (COL), MX?.1 (COL)
- net at MX?.2 (ROW): now also D?.2 (A) (x67)
- net COL4: now reaches MX?.1 (COL)
- net COL4: now also MX?.1 (COL), MX?.1 (COL), MX?.1 (COL)
- net COL5: now reaches MX?.1 (COL)
- net COL5: now also MX?.1 (COL), MX?.1 (COL), MX?.1 (COL)
- net COL6: now reaches MX?.1 (COL)
- net COL6: now also MX?.1 (COL), MX?.1 (COL), MX?.1 (COL), MX?.1 (COL)
- net COL7: now reaches MX?.1 (COL)
- net COL7: now also MX?.1 (COL), MX?.1 (COL), MX?.1 (COL)
- net COL8: now reaches MX?.1 (COL)
- net COL8: now also MX?.1 (COL), MX?.1 (COL), MX?.1 (COL)
- net COL9: now reaches MX?.1 (COL)
- net COL9: now also MX?.1 (COL), MX?.1 (COL), MX?.1 (COL)
- net COL10: now reaches MX?.1 (COL)
- net COL10: now also MX?.1 (COL), MX?.1 (COL), MX?.1 (COL), MX?.1 (COL)
- net COL11: now reaches MX?.1 (COL)
- net COL11: now also MX?.1 (COL), MX?.1 (COL), MX?.1 (COL), MX?.1 (COL)
- net COL12: now reaches MX?.1 (COL)
- net COL12: now also MX?.1 (COL), MX?.1 (COL), MX?.1 (COL), MX?.1 (COL)
- net COL13: now reaches MX?.1 (COL)
- net COL13: now also MX?.1 (COL), MX?.1 (COL)
- net COL14: now reaches MX?.1 (COL)
- net COL14: now also MX?.1 (COL), MX?.1 (COL), MX?.1 (COL), MX?.1 (COL)
- net COL2: now reaches MX?.1 (COL)
- net COL2: now also MX?.1 (COL), MX?.1 (COL), MX?.1 (COL), MX?.1 (COL)
- net COL1: now reaches MX?.1 (COL)
- net COL1: now also MX?.1 (COL), MX?.1 (COL), MX?.1 (COL), MX?.1 (COL)
- net COL0: now reaches MX?.1 (COL)
- net COL0: now also MX?.1 (COL), MX?.1 (COL), MX?.1 (COL), MX?.1 (COL)
- new net ROW0: D?.1 (K), D?.1 (K), D?.1 (K), D?.1 (K), D?.1 (K), D?.1 (K), D?.1 (K), D?.1 (K), D?.1 (K), D?.1 (K), D?.1 (K), D?.1 (K), D?.1 (K), D?.1 (K), D?.1 (K)
- new net ROW1: D?.1 (K), D?.1 (K), D?.1 (K), D?.1 (K), D?.1 (K), D?.1 (K), D?.1 (K), D?.1 (K), D?.1 (K), D?.1 (K), D?.1 (K), D?.1 (K), D?.1 (K), D?.1 (K), D?.1 (K)
- new net ROW2: D?.1 (K), D?.1 (K), D?.1 (K), D?.1 (K), D?.1 (K), D?.1 (K), D?.1 (K), D?.1 (K), D?.1 (K), D?.1 (K), D?.1 (K), D?.1 (K), D?.1 (K), D?.1 (K)
- new net ROW3: D?.1 (K), D?.1 (K), D?.1 (K), D?.1 (K), D?.1 (K), D?.1 (K), D?.1 (K), D?.1 (K), D?.1 (K), D?.1 (K), D?.1 (K), D?.1 (K), D?.1 (K), D?.1 (K)
- new net ROW4: D?.1 (K), D?.1 (K), D?.1 (K), D?.1 (K), D?.1 (K), D?.1 (K), D?.1 (K), D?.1 (K), D?.1 (K)
Other:
- moved on the sheet: MX?

Commit message: Complete schematic
Parts:
- added C1: 1u, Capacitor_SMD:C_0805_2012Metric_Pad1.15x1.40mm_HandSolder, symbol Device:C_Small
- added C2, C3: 22p, Capacitor_SMD:C_0805_2012Metric_Pad1.15x1.40mm_HandSolder, symbol Device:C_Small
- added C4, C5, C6, C7: 0.1u, Capacitor_SMD:C_0805_2012Metric_Pad1.15x1.40mm_HandSolder, symbol Device:C_Small
- added C8: 4.7u, Capacitor_SMD:C_0805_2012Metric_Pad1.15x1.40mm_HandSolder, symbol Device:C_Small
- added F1: 500mA, Fuse:Fuse_1206_3216Metric_Pad1.42x1.75mm_HandSolder, symbol Device:Polyfuse_Small
- added J1: USB4085-GF-A_REVA, USB4085-GF-A_REVA:GCT_USB4085-GF-A_REVA, symbol USB4085-GF-A_REVA:USB4085-GF-A_REVA
- added R1, R6: 10k, Resistor_SMD:R_0805_2012Metric_Pad1.15x1.40mm_HandSolder, symbol Device:R_Small
- added R2, R3: 22 ohm, Resistor_SMD:R_0805_2012Metric_Pad1.15x1.40mm_HandSolder, symbol Device:R_Small
- added R4, R5: 5.1k, Resistor_SMD:R_0805_2012Metric_Pad1.15x1.40mm_HandSolder, symbol Device:R_Small
- added SW1: SW_PUSH, Button_Switch_SMD:SW_SPST_TL3342, symbol keyboard_parts:SW_PUSH
- added U1: ATmega32U4-AU, Package_QFP:TQFP-44_10x10mm_P0.8mm, symbol MCU_Microchip_ATmega:ATmega32U4-AU
- added X1: XTAL_GND, Crystal:Crystal_SMD_SeikoEpson_FA238-4Pin_3.2x2.5mm_HandSoldering, symbol keyboard_parts:XTAL_GND
- D1, D10, D11, D12, D13, D14, D15, D16, D17, D18, D19, D2, D20, D21, D22, D23, D24, D25, D26, D27, D28, D29, D3, D30, D31, D32, D33, D34, D35, D36, D37, D38, D39, D4, D40, D41, D42, D43, D44, D45, D46, D47, D48, D49, D5, D50, D51, D52, D53, D54, D55, D56, D57, D58, D59, D6, D60, D61, D62, D63, D64, D65, D66, D67, D7, D8, D9: renamed from D?; footprint (none) -> Diode_SMD:D_SOD-123
- MX1, MX10, MX11, MX12, MX13, MX15, MX17, MX18, MX19, MX2, MX20, MX21, MX22, MX23, MX24, MX25, MX26, MX27, MX28, MX3, MX30, MX32, MX33, MX34, MX35, MX36, MX37, MX38, MX39, MX4, MX40, MX41, MX42, MX44, MX46, MX47, MX48, MX49, MX5, MX50, MX51, MX52, MX53, MX54, MX55, MX57, MX58, MX6, MX63, MX64, MX65, MX66, MX67, MX7, MX8, MX9: renamed from MX?; footprint (none) -> MX_Only:MXOnly-1U-NoLED
- MX14: renamed from MX?; footprint (none) -> MX_Only:MXOnly-2U-NoLED
- MX16, MX29: renamed from MX?; footprint (none) -> MX_Only:MXOnly-1.5U-NoLED
- MX31, MX59, MX60, MX61: renamed from MX?; footprint (none) -> MX_Only:MXOnly-1.25U-NoLED
- MX43, MX45: renamed from MX?; footprint (none) -> MX_Only:MXOnly-2.25U-NoLED
- MX56: renamed from MX?; footprint (none) -> MX_Only:MXOnly-1.75U-NoLED
- MX62: renamed from MX?; footprint (none) -> MX_Only:MXOnly-7U-ReversedStabilizers-NoLED
Connections:
- new net: U1.2 (UVCC), U1.24 (AVCC), U1.44 (AVCC)
- new net: R1.1, U1.33 (~HWB~/PE2)
- new net: C1.1, U1.6 (UCAP)
- new net: J1.A5 (CC1), R5.2
- new net: J1.A6 (DP1), J1.B6 (DP2), R3.2
- new net: J1.A7 (DN1), J1.B7 (DN2), R2.2
- new net: J1.B5 (CC2), R4.2
- new net +5V: C4.1, C5.1, C6.1, C7.1, C8.1, F1.2, R6.1, U1.14 (VCC), U1.34 (VCC), U1.7 (VBUS)
- new net D+: R3.1, U1.4 (D+)
- new net D-: R2.1, U1.3 (D-)
- new net GND: C1.2, C2.2, C3.2, C4.2, C5.2, C6.2, C7.2, C8.2, J1.A1 (GND), J1.A12 (GND), J1.B1 (GND), J1.B12 (GND), J1.P1 (SHELL), J1.P2 (SHELL), J1.P3 (SHELL), J1.P4 (SHELL), R1.2, R4.1, R5.1, SW1.1, U1.15 (GND), U1.23 (GND), U1.35 (GND), U1.43 (GND), U1.5 (UGND), X1.3
- new net RESET: R6.2, SW1.2, U1.13 (~RESET)
- new net VCC: F1.1, J1.A4 (VBUS), J1.A9 (VBUS), J1.B4 (VBUS), J1.B9 (VBUS)
- new net XTAL1: C2.1, U1.17 (XTAL1), X1.1
- new net XTAL2: C3.1, U1.16 (XTAL2), X1.2
- no-connect marks 0 -> 3
Other:
- note added: "Crystal"
- note added: "Decoupling Caps"
- note added: "Reset\n"
- note added: "USB-C 2.0\n\n"

Commit message: Place components
Parts:
- MX63: footprint MX_Only:MXOnly-1U-NoLED -> MX_Only:MXOnly-1.25U-NoLED
Changed lines of the file:
@@
 F 0 "MX63" H 9433 4623 60  0000 C CNN
 F 1 "MX-NoLED" H 9433 4549 20  0000 C CNN
-F 2 "MX_Only:MXOnly-1U-NoLED" H 8775 4375 60  0001 C CNN
+F 2 "MX_Only:MXOnly-1.25U-NoLED" H 8775 4375 60  0001 C CNN
 F 3 "" H 8775 4375 60  0001 C CNN
 	1    9400 4400
@@
 Wire Wire Line
 	10400 2500 10050 2500
-Wire Wire Line
-	10750 3250 10050 3250
 Connection ~ 5850 3250
 Wire Wire Line
@@
 Wire Wire Line
 	9700 3250 9350 3250
-Connection ~ 10050 3250
-Wire Wire Line
-	10050 3250 9700 3250
-Wire Wire Line
-	10750 4000 10050 4000
 Connection ~ 5850 4000
 Wire Wire Line
@@
 Wire Wire Line
 	9700 4000 9350 4000
-Connection ~ 10050 4000
-Wire Wire Line
-	10050 4000 9700 4000
 Wire Wire Line
 	10750 4750 10400 4750
@@
 Wire Wire Line
 	9900 3600 9900 2850
-Wire Wire Line
-	10250 4350 10250 3600
 Connection ~ 10250 1350
 Wire Wire Line
@@
 Wire Wire Line
 	10250 2100 10250 1350
-Connection ~ 10250 2850
-Wire Wire Line
-	10250 2850 10250 2100
-Connection ~ 10250 3600
-Wire Wire Line
-	10250 3600 10250 2850
-Wire Wire Line
-	10600 4350 10600 2100
 Connection ~ 10600 1350
 Wire Wire Line
@@
 	1    0    0    -1
 $EndComp
+Wire Wire Line
+	10250 2100 10250 2850
+Wire Wire Line
+	9700 4000 10050 4000
+Wire Wire Line
+	9700 3250 10050 3250
+Connection ~ 10250 2850
+Wire Wire Line
+	10250 2850 10250 3600
+Connection ~ 10050 3250
+Connection ~ 10250 3600
+Wire Wire Line
+	10250 3600 10250 4350
+Connection ~ 10050 4000
+Wire Wire Line
+	10050 3250 10750 3250
+Wire Wire Line
+	10050 4000 10750 4000
+Wire Wire Line
+	10600 2100 10600 4350
 $EndSCHEMATC

Commit message: Component placement
Parts:
- removed U1: ATmega32U4-AU, Package_QFP:TQFP-44_10x10mm_P0.8mm, symbol MCU_Microchip_ATmega:ATmega32U4-AU
- added U1: ATMEGA32U4, Package_QFP:TQFP-44_10x10mm_P0.8mm, symbol keyboard_parts:ATMEGA32U4
Connections:
- net +5V: now also U1.14 (VCC), U1.2 (UVcc), U1.24 (AVCC), U1.34 (VCC), U1.44 (AVCC), U1.7 (VBus)
- net D+: now also U1.4 (D+)
- net D-: now also U1.3 (D-)
- net GND: now also U1.15 (GND), U1.23 (GND), U1.35 (GND), U1.43 (GND), U1.5 (UGnd)
- net RESET: now also U1.13 (~RESET)
- net XTAL1: now also U1.16 (XTAL1)
- net XTAL2: now also U1.17 (XTAL2)
- net at R1.1: now also U1.33 (~HWB/PE2)
- net at C1.1: now also U1.6 (UCap)
- no-connect marks 3 -> 2
Other:
- note added: "@MEGA"
- moved on the sheet: C1, R1
Changed lines of the file:
@@
 Text GLabel 5600 4750 0    50   Input ~ 0
 ROW4
-$Comp
-L MCU_Microchip_ATmega:ATmega32U4-AU U1
-U 1 1 5F5682CF
-P 3450 3250
-F 0 "U1" H 2600 1700 50  0000 C CNN
-F 1 "ATmega32U4-AU" H 2600 1600 50  0000 C CNN
-F 2 "Package_QFP:TQFP-44_10x10mm_P0.8mm" H 3450 3250 50  0001 C CIN
-F 3 "http://ww1.microchip.com/downloads/en/DeviceDoc/Atmel-7766-8-bit-AVR-ATmega16U4-32U4_Datasheet.pdf" H 3450 3250 50  0001 C CNN
-	1    3450 3250
-	1    0    0    -1
-$EndComp
-Text GLabel 2850 1750 0    50   Input ~ 0
+Text GLabel 1700 3300 0    50   Input ~ 0
 RESET
 Text GLabel 6050 7350 2    50   Input ~ 0
@@
 $EndComp
 $Comp
-L power:GND #PWR0103
-U 1 1 5F57B366
-P 3600 5050
-F 0 "#PWR0103" H 3600 4800 50  0001 C CNN
-F 1 "GND" H 3600 5100 50  0000 C CNN
-F 2 "" H 3600 5050 50  0001 C CNN
-F 3 "" H 3600 5050 50  0001 C CNN
-	1    3600 5050
-	1    0    0    -1
-$EndComp
-Wire Wire Line
-	3350 5050 3450 5050
-Connection ~ 3450 5050
-Wire Wire Line
-	3450 5050 3600 5050
-Wire Wire Line
-	3350 1450 3350 1400
-Wire Wire Line
-	3350 1400 3550 1400
-Wire Wire Line
-	3550 1400 3550 1450
-$Comp
 L power:+5V #PWR0104
 U 1 1 5F588B35
-P 3450 1300
-F 0 "#PWR0104" H 3450 1150 50  0001 C CNN
-F 1 "+5V" H 3465 1473 50  0000 C CNN
-F 2 "" H 3450 1300 50  0001 C CNN
-F 3 "" H 3450 1300 50  0001 C CNN
-	1    3450 1300
-	1    0    0    -1
-$EndComp
-Wire Wire Line
-	3450 1300 3450 1450
+P 1600 2050
+F 0 "#PWR0104" H 1600 1900 50  0001 C CNN
+F 1 "+5V" H 1615 2223 50  0000 C CNN
+F 2 "" H 1600 2050 50  0001 C CNN
+F 3 "" H 1600 2050 50  0001 C CNN
+	1    1600 2050
+	1    0    0    -1
+$EndComp
+Wire Wire Line
+	1600 2050 1600 2200
 $Comp
 L keyboard_parts:XTAL_GND X1
@@
 Text GLabel 4300 7000 1    50   Input ~ 0
 XTAL2
-Text GLabel 2850 1950 0    50   Input ~ 0
+Text GLabel 1700 3600 0    50   Input ~ 0
 XTAL1
-Text GLabel 2850 2150 0    50   Input ~ 0
+Text GLabel 1700 3700 0    50   Input ~ 0
 XTAL2
-NoConn ~ 2850 2350
 $Comp
 L power:+5V #PWR0106
 U 1 1 5F5B165B
-P 2700 2550
-F 0 "#PWR0106" H 2700 2400 50  0001 C CNN
-F 1 "+5V" H 2715 2723 50  0000 C CNN
-F 2 "" H 2700 2550 50  0001 C CNN
-F 3 "" H 2700 2550 50  0001 C CNN
-	1    2700 2550
-	1    0    0    -1
-$EndComp
-Wire Wire Line
-	2700 2550 2850 2550
-Text GLabel 2850 2750 0    50   Input ~ 0
+P 1550 2700
+F 0 "#PWR0106" H 1550 2550 50  0001 C CNN
+F 1 "+5V" H 1565 2873 50  0000 C CNN
+F 2 "" H 1550 2700 50  0001 C CNN
+F 3 "" H 1550 2700 50  0001 C CNN
+	1    1550 2700
+	1    0    0    -1
+$EndComp
+Wire Wire Line
+	1550 2700 1700 2700
+Text GLabel 1700 2400 0    50   Input ~ 0
 D+
-Text GLabel 2850 2850 0    50   Input ~ 0
+Text GLabel 1700 2300 0    50   Input ~ 0
 D-
 $Comp
 L Device:R_Small R1
 U 1 1 5F5B953F
-P 4200 3850
-F 0 "R1" V 4396 3850 50  0000 C CNN
-F 1 "10k" V 4305 3850 50  0000 C CNN
-F 2 "Resistor_SMD:R_0805_2012Metric_Pad1.15x1.40mm_HandSolder" H 4200 3850 50  0001 C CNN
-F 3 "~" H 4200 3850 50  0001 C CNN
-	1    4200 3850
+P 4000 3200
+F 0 "R1" V 4196 3200 50  0000 C CNN
+F 1 "10k" V 4105 3200 50  0000 C CNN
+F 2 "Resistor_SMD:R_0805_2012Metric_Pad1.15x1.40mm_HandSolder" H 4000 3200 50  0001 C CNN
+F 3 "~" H 4000 3200 50  0001 C CNN
+	1    4000 3200
 	0    -1   -1   0
 $EndComp
 Wire Wire Line
-	4100 3850 4050 3850
+	3900 3200 3850 3200
 $Comp
 L power:GND #PWR0107
 U 1 1 5F5C1E45
-P 4350 3850
-F 0 "#PWR0107" H 4350 3600 50  0001 C CNN
-F 1 "GND" H 4355 3677 50  0000 C CNN
-F 2 "" H 4350 3850 50  0001 C CNN
-F 3 "" H 4350 3850 50  0001 C CNN
-	1    4350 3850
-	1    0    0    -1
-$EndComp
-Wire Wire Line
-	4350 3850 4300 3850
+P 4150 3200
+F 0 "#PWR0107" H 4150 2950 50  0001 C CNN
+F 1 "GND" H 4155 3027 50  0000 C CNN
+F 2 "" H 4150 3200 50  0001 C CNN
+F 3 "" H 4150 3200 50  0001 C CNN
+	1    4150 3200
+	1    0    0    -1
+$EndComp
+Wire Wire Line
+	4150 3200 4100 3200
 $Comp
 L Device:C_Small C1
 U 1 1 5F5CAA76
-P 2600 3050
-F 0 "C1" V 2371 3050 50  0000 C CNN
-F 1 "1u" V 2462 3050 50  0000 C CNN
-F 2 "Capacitor_SMD:C_0805_2012Metric_Pad1.15x1.40mm_HandSolder" H 2600 3050 50  0001 C CNN
-F 3 "~" H 2600 3050 50  0001 C CNN
-	1    2600 3050
+P 1450 2600
+F 0 "C1" V 1221 2600 50  0000 C CNN
+F 1 "1u" V 1312 2600 50  0000 C CNN
+F 2 "Capacitor_SMD:C_0805_2012Metric_Pad1.15x1.40mm_HandSolder" H 1450 2600 50  0001 C CNN
+F 3 "~" H 1450 2600 50  0001 C CNN
+	1    1450 2600
 	0    1    1    0
 $EndComp
@@
 L power:GND #PWR0108
 U 1 1 5F5DFA66
-P 2450 3050
-F 0 "#PWR0108" H 2450 2800 50  0001 C CNN
-F 1 "GND" H 2455 2877 50  0000 C CNN
-F 2 "" H 2450 3050 50  0001 C CNN
-F 3 "" H 2450 3050 50  0001 C CNN
-	1    2450 3050
-	1    0    0    -1
-$EndComp
-Wire Wire Line
-	2450 3050 2500 3050
-Wire Wire Line
-	2700 3050 2850 3050
+P 1300 2600
+F 0 "#PWR0108" H 1300 2350 50  0001 C CNN
+F 1 "GND" H 1305 2427 50  0000 C CNN
+F 2 "" H 1300 2600 50  0001 C CNN
+F 3 "" H 1300 2600 50  0001 C CNN
+	1    1300 2600
+	1    0    0    -1
+$EndComp
+Wire Wire Line
+	1300 2600 1350 2600
+Wire Wire Line
+	1550 2600 1700 2600
 Text Notes 3700 6600 0    118  ~ 24
 Crystal
@@
 Wire Wire Line
 	10600 2100 10600 4350
+$Comp
+L keyboard_parts:ATMEGA32U4 U1
+U 1 1 5F56E3DD
+P 2750 3150
+F 0 "U1" H 2775 4487 60  0000 C CNN
+F 1 "ATMEGA32U4" H 2775 4381 60  0000 C CNN
+F 2 "Package_QFP:TQFP-44_10x10mm_P0.8mm" H 2750 3150 60  0001 C CNN
+F 3 "" H 2750 3150 60  0000 C CNN
+	1    2750 3150
+	1    0    0    -1
+$EndComp
+Wire Wire Line
+	1700 2200 1600 2200
+$Comp
+L power:+5V #PWR0103
+U 1 1 5F5A8F73
+P 1350 3400
+F 0 "#PWR0103" H 1350 3250 50  0001 C CNN
+F 1 "+5V" H 1365 3573 50  0000 C CNN
+F 2 "" H 1350 3400 50  0001 C CNN
+F 3 "" H 1350 3400 50  0001 C CNN
+	1    1350 3400
+	1    0    0    -1
+$EndComp
+$Comp
+L power:GND #PWR0116
+U 1 1 5F5AA002
+P 1350 3500
+F 0 "#PWR0116" H 1350 3250 50  0001 C CNN
+F 1 "GND" H 1355 3327 50  0000 C CNN
+F 2 "" H 1350 3500 50  0001 C CNN
+F 3 "" H 1350 3500 50  0001 C CNN
+	1    1350 3500
+	1    0    0    -1
+$EndComp
+Wire Wire Line
+	1350 3500 1700 3500
+Wire Wire Line
+	1700 3400 1350 3400
+Wire Wire Line
+	1700 2500 1300 2500
+Wire Wire Line
+	1300 2500 1300 2600
+Connection ~ 1300 2600
+Text Notes 2450 1600 0    118  ~ 24
+@MEGA
+$Comp
+L power:+5V #PWR?
+U 1 1 5F61FD1D
+P 4000 2100
+F 0 "#PWR?" H 4000 1950 50  0001 C CNN
+F 1 "+5V" H 4015 2273 50  0000 C CNN
+F 2 "" H 4000 2100 50  0001 C CNN
+F 3 "" H 4000 2100 50  0001 C CNN
+	1    4000 2100
+	1    0    0    -1
+$EndComp
+$Comp
+L power:GND #PWR?
+U 1 1 5F620425
+P 4000 2200
+F 0 "#PWR?" H 4000 1950 50  0001 C CNN
+F 1 "GND" H 4005 2027 50  0000 C CNN
+F 2 "" H 4000 2200 50  0001 C CNN
+F 3 "" H 4000 2200 50  0001 C CNN
+	1    4000 2200
+	1    0    0    -1
+$EndComp
+Wire Wire Line
+	4000 2200 3850 2200
+Wire Wire Line
+	4000 2100 3850 2100
+$Comp
+L power:GND #PWR?
+U 1 1 5F635EFD
+P 4450 3000
+F 0 "#PWR?" H 4450 2750 50  0001 C CNN
+F 1 "GND" H 4455 2827 50  0000 C CNN
+F 2 "" H 4450 3000 50  0001 C CNN
+F 3 "" H 4450 3000 50  0001 C CNN
+	1    4450 3000
+	1    0    0    -1
+$EndComp
+$Comp
+L power:+5V #PWR?
+U 1 1 5F636303
+P 4300 3100
+F 0 "#PWR?" H 4300 2950 50  0001 C CNN
+F 1 "+5V" H 4315 3273 50  0000 C CNN
+F 2 "" H 4300 3100 50  0001 C CNN
+F 3 "" H 4300 3100 50  0001 C CNN
+	1    4300 3100
+	1    0    0    -1
+$EndComp
+Wire Wire Line
+	4300 3100 3850 3100
+Wire Wire Line
+	3850 3000 4450 3000
+$Comp
+L power:+5V #PWR?
+U 1 1 5F64C6D1
+P 4000 4100
+F 0 "#PWR?" H 4000 3950 50  0001 C CNN
+F 1 "+5V" H 4015 4273 50  0000 C CNN
+F 2 "" H 4000 4100 50  0001 C CNN
+F 3 "" H 4000 4100 50  0001 C CNN
+	1    4000 4100
+	1    0    0    -1
+$EndComp
+$Comp
+L power:GND #PWR?
+U 1 1 5F64CD40
+P 4000 4200
+F 0 "#PWR?" H 4000 3950 50  0001 C CNN
+F 1 "GND" H 4005 4027 50  0000 C CNN
+F 2 "" H 4000 4200 50  0001 C CNN
+F 3 "" H 4000 4200 50  0001 C CNN
+	1    4000 4200
+	1    0    0    -1
+$EndComp
+Wire Wire Line
+	4000 4200 3850 4200
+Wire Wire Line
+	3850 4100 4000 4100
 $EndSCHEMATC

Commit message: Route traces
Connections:
- net COL0: now also U1.40 (PF1)
- net COL1: now also U1.39 (PF4)
- net COL10: now also U1.21 (PD3/TXD1)
- net COL11: now also U1.20 (PD2/RXD1)
- net COL12: now also U1.19 (PD1/INT1)
- net COL13: now also U1.12 (PB7/~RTS)
- net COL14: now also U1.18 (PD0/INT0)
- net COL2: now also U1.38 (PF5)
- net COL3: now also U1.37 (PF6)
- net COL4: now also U1.36 (PF7)
- net COL5: now also U1.32 (PC7)
- net COL6: now also U1.31 (PC6)
- net COL7: now also U1.41 (PF0)
- net COL8: now also U1.25 (ICP1/PD4)
- net COL9: now also U1.22 (PD5/XCK1)
- net ROW0: now also U1.26 (T1/PD6)
- net ROW1: now also U1.27 (T0/PD7)
- net ROW2: now also U1.28 (PB4)
- net ROW3: now also U1.29 (PB5)
- net ROW4: now also U1.30 (PB6)
Changed lines of the file:
@@
 Wire Wire Line
 	3850 4100 4000 4100
+Text GLabel 3850 3500 2    50   Input ~ 0
+ROW4
+Text GLabel 3850 3600 2    50   Input ~ 0
+ROW3
+Text GLabel 3850 3800 2    50   Input ~ 0
+ROW1
+Text GLabel 3850 3900 2    50   Input ~ 0
+ROW0
+Text GLabel 3850 2400 2    50   Input ~ 0
+COL7
+Text GLabel 3850 3400 2    50   Input ~ 0
+COL6
+Text GLabel 3850 3300 2    50   Input ~ 0
+COL5
+Text GLabel 3850 2900 2    50   Input ~ 0
+COL4
+Text GLabel 3850 2800 2    50   Input ~ 0
+COL3
+Text GLabel 3850 2700 2    50   Input ~ 0
+COL2
+Text GLabel 3850 3700 2    50   Input ~ 0
+ROW2
+Text GLabel 3850 2600 2    50   Input ~ 0
+COL1
+Text GLabel 3850 2500 2    50   Input ~ 0
+COL0
+Text GLabel 3850 4000 2    50   Input ~ 0
+COL8
+Text GLabel 1700 4200 0    50   Input ~ 0
+COL9
+Text GLabel 1700 4100 0    50   Input ~ 0
+COL10
+Text GLabel 1700 4000 0    50   Input ~ 0
+COL11
+Text GLabel 1700 3900 0    50   Input ~ 0
+COL12
+Text GLabel 1700 3800 0    50   Input ~ 0
+COL14
+Text GLabel 1700 3200 0    50   Input ~ 0
+COL13
 $EndSCHEMATC

Commit message: PCB
Parts:
- removed D15, D29, D30, D44, D48, D49, D51, D52, D53, D58, D59, D60, D61, D62, D63, D64, D65, D66, D67: 22p, Diode_SMD:D_SOD-123, symbol Device:D_Small
- removed MX15, MX30, MX44, MX48, MX49, MX51, MX52, MX53, MX58, MX64, MX65, MX66, MX67: MX-NoLED, MX_Only:MXOnly-1U-NoLED, symbol MX_Alps_Hybrid:MX-NoLED
- removed MX29: MX-NoLED, MX_Only:MXOnly-1.5U-NoLED, symbol MX_Alps_Hybrid:MX-NoLED
- removed MX59, MX60, MX61, MX63: MX-NoLED, MX_Only:MXOnly-1.25U-NoLED, symbol MX_Alps_Hybrid:MX-NoLED
- removed MX62: MX-NoLED, MX_Only:MXOnly-7U-ReversedStabilizers-NoLED, symbol MX_Alps_Hybrid:MX-NoLED
- MX14: footprint MX_Only:MXOnly-2U-NoLED -> MX_Only:MXOnly-1U-NoLED
- MX16: footprint MX_Only:MXOnly-1.5U-NoLED -> MX_Only:MXOnly-1.25U-NoLED
- MX27: footprint MX_Only:MXOnly-1U-NoLED -> MX_Only:MXOnly-1.75U-NoLED
- MX31: footprint MX_Only:MXOnly-1.25U-NoLED -> MX_Only:MXOnly-1.75U-NoLED
- MX41, MX47, MX54: footprint MX_Only:MXOnly-1U-NoLED -> MX_Only:MXOnly-1.25U-NoLED
- MX43: footprint MX_Only:MXOnly-2.25U-NoLED -> MX_Only:MXOnly-1U-NoLED
- MX45: footprint MX_Only:MXOnly-2.25U-NoLED -> MX_Only:MXOnly-1.25U-NoLED
- MX50: footprint MX_Only:MXOnly-1U-NoLED -> MX_Only:MXOnly-6.25U-ReversedStabilizers-NoLED
- MX56: footprint MX_Only:MXOnly-1.75U-NoLED -> MX_Only:MXOnly-1U-NoLED
Connections:
- net COL14: no longer names the net of U1.18 (PD0/INT0)
- net ROW4: no longer names the net of U1.30 (PB6)
